File: Hardware/PCBs/MainBoard/STARGLIDER_MainBoard_rev1/STARGLIDER_MainBoard_rev1.kicad_pcb (KiCad board)
At the start: 4 copper layers, 60 x 60 mm, 71 parts, among them J1 USB_C_Receptacle_USB2.0, J2 Micro_SD_Card, Q1 NMOS, Q2 NMOS, U1 STM32G474RETx, U2 AMS1117-5.0, U3 AMS1117-3.3, U4 USBLC6-2SC6, U5 MPU-6050, U6 BME280, U7 LSM6DS3, X1 24Mhz, X2 32.768KHz

Commit message: V0.1
Other:
- board text added: "Main Board"

Commit message: Main Board rev1 done
Parts:
- removed NT1: NetTie_2, NetTie:NetTie-2_SMD_Pad0.5mm
- added R13: 10K, Resistor_SMD:R_0603_1608Metric, B.Cu at (113.7, 103.0)
- added R14: 10K, Resistor_SMD:R_0603_1608Metric, B.Cu at (112.1, 106.2)
- 2x_BME280_SPI1: renamed from 2x BME280
- 3x_PWM1: renamed from 3x PWM
- D1, D2: footprint Diode_SMD:D_0805_2012Metric -> Diode_SMD:D_SOD-123
- moved C3 1.23 mm to (100.0, 113.5), turned to -90 degrees
- moved C4 1.06 mm to (98.3, 113.5), turned to -90 degrees
- moved D1 0.29 mm to (127.1, 91.0)
- renumbered Buzzer to BZ1, GPIOB to GPIOB1, GPIOC to GPIOC1, LPUART to LPUART1, SWD to PROG1, -POWER+ to Power1, NRST to SW2
Connections:
- C6 pad 2: GNDA -> GND
- C7 pad 2: GNDA -> GND
- U1 pad 27: GNDA -> GND
Routing:
- net +3V3: track 104.3 -> 123.5 mm, vias 19 -> 10
- net GNDA: track 10.8 -> 0.00 mm
- net GND: track 154.3 -> 165.0 mm, vias 50 -> 51
- net I2C3_SCL: track 12.2 -> 14.0 mm
- net +5V: track 33.4 -> 31.9 mm, vias 6 -> 5
- net I2C3_SDA: track 14.4 -> 15.9 mm
- net VDC: track 20.8 -> 19.9 mm
- net Net-(D1-A): track 3.97 -> 3.14 mm
Other:
- board text added: "-POWER+"
- board text added: "2x BME280"
- board text added: "3x PWM"
- board text added: "BOOT"
- board text added: "Buzzer"
- board text added: "GPIOB"
- board text added: "GPIOC"
- board text added: "JLCJLCJLCJLC"
- board text added: "LPUART"
- board text added: "NRST"
- board text added: "PROG"
- board text added: "RGB"
- board text added: "SPI3"
- board text added: "SWD"
- board text added: "USB"
