File: Hardware/PCBs/MainBoard/STARGLIDER_MainBoard_rev1/STARGLIDER_MainBoard_rev1.kicad_sch (KiCad schematic)
At the start: 66 parts, among them J1 USB_C_Receptacle_USB2.0, J2 Micro_SD_Card, Q1 NMOS, Q2 NMOS, SW1 SW_DPDT_x2, SW2 SW_SPST, U1 STM32G474RETx, U2 AMS1117-5.0, U3 AMS1117-3.3, U4 USBLC6-2SC6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

Commit message: Main Board rev1 done
Parts:
- removed NT1: NetTie_2, NetTie:NetTie-2_SMD_Pad0.5mm, symbol Device:NetTie_2
- added R13, R14: 10K, Resistor_SMD:R_0603_1608Metric, symbol Device:R
- D1, D2: footprint (none) -> Diode_SMD:D_SOD-123
- renumbered D2 to D3
Connections:
- net GNDA is gone; now on net GND: C6.2, C7.2, U1.27 (VSSA)
- net +3V3: now also R13.1, R14.1
- net I2C3_SCL: now also R14.2
- net I2C3_SDA: now also R13.2
